File: board-clima-esp32.kicad_sch (KiCad schematic)
At the start: 7 parts, among them IC1 ESP32-S3-WROOM-1-N8R8, J1 USB_C_Receptacle_USB2.0, U1 AMS1117-3.3

Commit message: edits
Parts:
- added C3: 1u, symbol Device:C
- added R3: 10k, symbol Device:R
- added SW1: RESET, symbol Switch:SW_Push
Connections:
- net GND: now also IC1.1 (GND_1), C3.2, SW1.1
- net USB+: now also IC1.14 (IO20)
- net USB-: now also IC1.13 (IO19)
- net +3V3: now reaches IC1.2 (3V3)
- net +3V3: now also R3.1
- net BOOT: now reaches IC1.27 (IO0)
- net at IC1.3 (EN): now also C3.1, R3.2, SW1.2
- net JTAG_TCK: now reaches IC1.32 (IO39)
- net JTAG_TDO: now reaches IC1.33 (IO40)
- net JTAG_TDI: now reaches IC1.34 (IO41)
- net JTAG_TMS: now reaches IC1.35 (IO42)
- net UART_RX: now reaches IC1.36 (RXD0)
- net UART_TX: now reaches IC1.37 (TXD0)

Commit message: sensor, relay sym footprint
Parts:
- added C4: 100n, symbol Device:C
- added D1: MRA4007T3G, Diode_SMD:D_SMA, symbol Diode:MRA4007T3G
- added D2, D3: LED, symbol Device:LED
- added HM1: BME280, BME280, symbol BME280:BME280
- added J2: Screw_Terminal_01x03, symbol Connector:Screw_Terminal_01x03
- added J3, J4: Conn_01x04_Pin, symbol Connector:Conn_01x04_Pin
- added J5: Conn_01x04_Pin, symbol Connector:Conn_01x03_Pin
- added J6: Conn_01x02_Pin, symbol Connector:Conn_01x02_Pin
- added Q1: 2N7002K, Package_TO_SOT_SMD:SOT-23, symbol Transistor_FET:2N7002K
- added R4, R5: 220, symbol Device:R
- added U2: ~, symbol JZC-32F:JZC-32F/C
- IC1: value ESP32-S3-WROOM-1-N8R8 -> ESP32-S3-WROOM-1-N8
Connections:
- net +3V3 is gone; now on net +3.3V: IC1.2 (3V3), R3.1
- net GND is gone; now on net +3.3V: C1.2, C2.2, C3.2, IC1.1 (GND_1), J1.A1 (GND), J1.A12 (GND), J1.B1 (GND), J1.B12 (GND), J1.S1 (SHIELD), R1.2, R2.2, SW1.1, U1.1 (GND)
- net +3.3V: now also IC1.40 (GND_2), IC1.41 (GND_3), IC1.42 (GND_4), IC1.43 (GND_5), IC1.44 (GND_6), IC1.45 (GND_7), IC1.46 (GND_8), IC1.47 (GND_9), IC1.48 (GND_10), IC1.49 (GND_11), C4.1, C4.2, D3.1 (K), HM1.1 (GND_1), HM1.2 (CSB), HM1.5 (SDO), HM1.6 (VDDIO), HM1.7 (GND_2), HM1.8 (VDD), J3.1 (Pin_1), J3.4 (Pin_4), J5.1 (Pin_1), J5.3 (Pin_3), J6.1 (Pin_1), Q1.2 (S), R5.1
- net BOOT: now also J6.2 (Pin_2)
- net JTAG_TCK: now also J4.4 (Pin_4)
- net JTAG_TDI: now also J4.2 (Pin_2)
- net JTAG_TDO: now also J4.3 (Pin_3)
- net JTAG_TMS: now also J4.1 (Pin_1)
- net UART_RX: now also J3.2 (Pin_2)
- net UART_TX: now also J3.3 (Pin_3)
- net SDA: now reaches IC1.18 (IO10)
- net SDA: now also HM1.3 (SDI)
- net SCK: now reaches IC1.19 (IO11)
- net SCK: now also HM1.4 (SCK)
- net RELAY: now reaches IC1.23 (IO21)
- net RELAY: now also Q1.1 (G)
- net GPIO38: now reaches IC1.31 (IO38)
- net GPIO38: now also J5.2 (Pin_2)
- net VBUS renamed +5V
- net +5V: now also D1.1 (K), R4.1, U2.1 (C1)
- new net: J2.1 (Pin_1), U2.5 (NO)
- new net: J2.2 (Pin_2), U2.3 (COM)
- new net: J2.3 (Pin_3), U2.4 (NC)
- new net: D2.2 (A), R4.2
- new net: D1.2 (A), D2.1 (K), Q1.3 (D), U2.2 (C2)
- new net: D3.2 (A), R5.2
- no-connect marks 3 -> 25
Other:
- note added: "Additional GPIO"
- note added: "BOOT Selector"
- note added: "JTAG"
- note added: "JZC-32F/C Relay"
- note added: "MCU"
- note added: "PSRAM"
- note added: "Power"
- note added: "Power LED"
- note added: "Relay Status LED"
- note added: "Temperature Sensor"
- note added: "UART"
- note added: "USB In"
- moved on the sheet: C1, C2, J1, R1, R2

Commit message: schematic ok
Parts:
- removed J6: Conn_01x02_Pin, symbol Connector:Conn_01x02_Pin
- added F1: Polyfuse, Fuse:Fuse_1812_4532Metric_Pad1.30x3.40mm_HandSolder, symbol Device:Polyfuse
- added R6, R7: 5.1k, Resistor_SMD:R_0805_2012Metric, symbol Device:R
- added R8: 10k, Resistor_SMD:R_0805_2012Metric, symbol Device:R
- added R9: 220, Resistor_SMD:R_0805_2012Metric, symbol Device:R
- added SW2: BOOT, Button_Switch_SMD:SW_Push_SPST_NO_Alps_SKRK, symbol Switch:SW_Push
- C1, C2, C3, C4: footprint (none) -> Capacitor_SMD:C_0805_2012Metric
- D2, D3: footprint (none) -> LED_SMD:LED_0805_2012Metric
- HM1: footprint BME280 -> BME280:BME280
- IC1: footprint ESP32S3WROOM1N8R8 -> ESP32-S3-WROOM-N8R8:ESP32S3WROOM1N8R8
- J1: footprint (none) -> USBC-31M12:HRO_TYPE-C-31-M-12
- J2: footprint (none) -> TerminalBlock:TerminalBlock_bornier-3_P5.08mm
- J3, J4, J5: footprint (none) -> Connector_PinHeader_2.54mm:PinHeader_1x04_P2.54mm_Vertical
- R1, R2, R3, R4, R5: footprint (none) -> Resistor_SMD:R_0805_2012Metric
- SW1: footprint (none) -> Button_Switch_SMD:SW_Push_SPST_NO_Alps_SKRK
- U2: value ~ -> JZC-32F/C; footprint (none) -> JZC-32FC:JZC-32FC
Connections:
- net +3.3V: now also R6.1, R7.1, R8.2, SW2.2
- net +5V: now also F1.2; no longer J1.A4 (VBUS), J1.A9 (VBUS), J1.B4 (VBUS), J1.B9 (VBUS)
- net BOOT: now also SW2.1
- net RELAY: now also R8.1, R9.1; no longer Q1.1 (G)
- net SCK: now also R7.2
- net SDA: now also R6.2
- new net: F1.1, J1.A4 (VBUS), J1.A9 (VBUS), J1.B4 (VBUS), J1.B9 (VBUS)
- new net: Q1.1 (G), R9.2
Other:
- note added: "Boot Selector"
- note added: "I2C PUN DNP"
- note removed: "BOOT Selector"
- note removed: "JZC-32F/C Relay"
- moved on the sheet: C4, D1, D2, HM1, J2, Q1, R4

Commit message: fucking via clearences
Parts:
- removed J1: USB_C_Receptacle_USB2.0, USBC-31M12:HRO_TYPE-C-31-M-12, symbol Connector:USB_C_Receptacle_USB2.0
- added J6: USB_C_Receptacle, USBC-31M12:HRO_TYPE-C-31-M-12, symbol Connector:USB_C_Receptacle
- J5: value Conn_01x04_Pin -> Conn_01x03_Pin; footprint Connector_PinHeader_2.54mm:PinHeader_1x04_P2.54mm_Vertical -> Connector_PinHeader_2.54mm:PinHeader_1x03_P2.54mm_Vertical
Connections:
- net +3.3V: no longer C1.2, C2.2, C3.2, C4.2, D3.1 (K), HM1.1 (GND_1), HM1.5 (SDO), HM1.7 (GND_2), IC1.1 (GND_1), IC1.40 (GND_2), IC1.41 (GND_3), IC1.42 (GND_4), IC1.43 (GND_5), IC1.44 (GND_6), IC1.45 (GND_7), IC1.46 (GND_8), IC1.47 (GND_9), IC1.48 (GND_10), IC1.49 (GND_11), J3.1 (Pin_1), J5.1 (Pin_1), Q1.2 (S), R1.2, R2.2, R8.2, SW1.1, SW2.2, U1.1 (GND)
- net USB+: now also J6.A6 (D+), J6.B6 (D+)
- net USB-: now also J6.A7 (D-), J6.B7 (D-)
- net at R2.1: now also J6.B5 (CC2)
- net at F1.1: now also J6.A4 (VBUS), J6.A9 (VBUS), J6.B4 (VBUS), J6.B9 (VBUS)
- net at R1.1: now also J6.A5 (CC1)
- new net GND: C1.2, C2.2, C3.2, C4.2, D3.1 (K), HM1.1 (GND_1), HM1.5 (SDO), HM1.7 (GND_2), IC1.1 (GND_1), IC1.40 (GND_2), IC1.41 (GND_3), IC1.42 (GND_4), IC1.43 (GND_5), IC1.44 (GND_6), IC1.45 (GND_7), IC1.46 (GND_8), IC1.47 (GND_9), IC1.48 (GND_10), IC1.49 (GND_11), J3.1 (Pin_1), J5.1 (Pin_1), J6.A1 (GND), J6.A12 (GND), J6.B1 (GND), J6.B12 (GND), J6.S1 (SHIELD), Q1.2 (S), R1.2, R2.2, R8.2, SW1.1, SW2.2, U1.1 (GND)
- no-connect marks 25 -> 33
Other:
- moved on the sheet: D1, D2, F1, J2, Q1, R1, R2, R4, R8, R9, U2

Commit message: should be done
Parts:
- added H1, H2: MountingHole, symbol Mechanical:MountingHole
Connections:
- net RELAY: now also IC1.16 (IO46); no longer IC1.23 (IO21)
Changed lines of the file:
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@@
   (no_connect (at 143.51 44.45))
   (no_connect (at 46.355 80.645))
-  (no_connect (at 143.51 67.31))
+  (no_connect (at 143.51 85.09))
   (no_connect (at 46.355 103.505))
   (no_connect (at 143.51 64.77))
@@
     (stroke (width 0) (type default))
   )
-  (wire (pts (xy 132.08 85.09) (xy 143.51 85.09))
+  (wire (pts (xy 132.08 67.31) (xy 143.51 67.31))
     (stroke (width 0) (type default))
   )
@@
     (effects (font (size 1.27 1.27)) (justify left bottom))
   )
-  (label "RELAY" (at 132.08 85.09 0) (fields_autoplaced)
+  (label "RELAY" (at 132.08 67.31 0) (fields_autoplaced)
     (effects (font (size 1.27 1.27)) (justify left bottom))
   )
@@
     )
   )
+  (symbol (lib_id "Mechanical:MountingHole") (at 266.7 145.415 0) (unit 1)
+    (in_bom yes) (on_board yes) (dnp no) (fields_autoplaced)
+    (property "Reference" "H2" (at 269.875 144.145 0)
+      (effects (font (size 1.27 1.27)) (justify left))
+    )
+    (property "Value" "MountingHole" (at 269.875 146.685 0)
+      (effects (font (size 1.27 1.27)) (justify left))
+    )
+    (property "Footprint" "" (at 266.7 145.415 0)
+      (effects (font (size 1.27 1.27)) hide)
+    )
+    (property "Datasheet" "~" (at 266.7 145.415 0)
+      (effects (font (size 1.27 1.27)) hide)
+    )
+    (instances
+      (project "board-clima-esp32"
+        (path "/ec184202-d4fa-4f1f-9fe7-c32d14dd4c20"
+          (reference "H2") (unit 1)
+        )
+      )
+    )
+  )
   (symbol (lib_id "Device:C") (at 125.73 134.62 0) (unit 1)
     (in_bom yes) (on_board yes) (dnp no) (fields_autoplaced)
@@
         )
       )
+    )
+  )
+  (symbol (lib_id "Mechanical:MountingHole") (at 266.7 139.065 0) (unit 1)
+    (in_bom yes) (on_board yes) (dnp no) (fields_autoplaced)
+    (property "Reference" "H1" (at 269.875 137.795 0)
+      (effects (font (size 1.27 1.27)) (justify left))
+    )
+    (property "Value" "MountingHole" (at 269.875 140.335 0)
+      (effects (font (size 1.27 1.27)) (justify left))
+    )
+    (property "Footprint" "" (at 266.7 139.065 0)
+      (effects (font (size 1.27 1.27)) hide)
+    )
+    (property "Datasheet" "~" (at 266.7 139.065 0)
+      (effects (font (size 1.27 1.27)) hide)
+    )
+    (instances
+      (project "board-clima-esp32"
+        (path "/ec184202-d4fa-4f1f-9fe7-c32d14dd4c20"
+          (reference "H1") (unit 1)
+        )
+      )

Commit message: editing stuff again
Parts:
- added J1: Conn_01x02_Pin, Connector_PinHeader_2.54mm:PinHeader_1x02_P2.54mm_Vertical, symbol Connector:Conn_01x02_Pin
- H1, H2: footprint (none) -> MountingHole:MountingHole_2.5mm
- J4: footprint Connector_PinHeader_2.54mm:PinHeader_1x04_P2.54mm_Vertical -> Connector_PinHeader_1.00mm:PinHeader_1x05_P1.00mm_Vertical; symbol Connector:Conn_01x04_Pin -> Connector:Conn_01x05_Pin
- J5: value Conn_01x03_Pin -> Conn_01x04_Pin; footprint Connector_PinHeader_2.54mm:PinHeader_1x03_P2.54mm_Vertical -> Connector_PinHeader_2.54mm:PinHeader_1x04_P2.54mm_Vertical; symbol Connector:Conn_01x03_Pin -> Connector:Conn_01x04_Pin
Connections:
- net +3.3V: now also J5.4 (Pin_4); no longer J5.3 (Pin_3)
- net GND: now also J4.1 (Pin_1)
- net JTAG_TMS: now also J4.5 (Pin_5); no longer J4.1 (Pin_1)
- net SCK: now also J1.1 (Pin_1)
- net SDA: now also J1.2 (Pin_2)
- net GPIO2: now reaches IC1.38 (IO2)
- net GPIO2: now also J5.2 (Pin_2)
- net GPIO1: now reaches IC1.39 (IO1)
- net GPIO1: now also J5.3 (Pin_3)
- net GPIO38: no longer names the net of IC1.31 (IO38)
- net GPIO38: no longer J5.2 (Pin_2)
- no-connect marks 33 -> 32
Other:
- moved on the sheet: H1, H2, J3, SW2

Commit message: edit to get jlc assembly
Parts:
- removed D1: MRA4007T3G, Diode_SMD:D_SMA, symbol Diode:MRA4007T3G
- removed Q1: 2N7002K, Package_TO_SOT_SMD:SOT-23, symbol Transistor_FET:2N7002K
- added D1: SM4007, Diode_SMD:D_MELF, symbol Diode:SM4007
- added Q1: AO3400A, Package_TO_SOT_SMD:SOT-23, symbol Transistor_FET:AO3400A
- C1, C2: LCSC (none) -> C15850
- C3: LCSC (none) -> C28323
- C4: LCSC (none) -> C49678
- D2, D3: LCSC (none) -> C84256
- F1: LCSC (none) -> C960026
- HM1: LCSC (none) -> C92489
- IC1: value ESP32-S3-WROOM-1-N8 -> ESP32-S3-WROOM-1-N4; LCSC (none) -> C2913197
- J1: footprint Connector_PinHeader_2.54mm:PinHeader_1x02_P2.54mm_Vertical -> Connector_PinHeader_2.54mm:PinHeader_1x03_P2.54mm_Vertical; symbol Connector:Conn_01x02_Pin -> Connector:Conn_01x03_Pin
- J6: LCSC (none) -> C165948
- R1, R2, R6, R7: LCSC (none) -> C17673
- R3, R8: LCSC (none) -> C17414
- R4, R5, R9: LCSC (none) -> C17557
- SW1, SW2: footprint Button_Switch_SMD:SW_Push_SPST_NO_Alps_SKRK -> Button_Switch_SMD:SW_Push_1P1T_XKB_TS-1187A; LCSC (none) -> C318884
- U1: LCSC (none) -> C6186
Connections:
- net +5V: now also D1.1 (K)
- net GND: now also J1.1 (Pin_1), Q1.2 (S)
- net SCK: now also J1.2 (Pin_2); no longer J1.1 (Pin_1)
- net SDA: now also J1.3 (Pin_3); no longer J1.2 (Pin_2)
- net at D2.1 (K), U2.2 (C2): now also D1.2 (A), Q1.3 (D)
- net at R9.2: now also Q1.1 (G)
Other:
- note added: "Additional I2C"
- moved on the sheet: D2, J2, J3, J4, R4, R8, R9, U2

Commit message: component edits, terminalblock footprint
Parts:
- C1, C2: Manufacturer_Part_Number (none) -> CL21A106KAYNNNE
- C3: Manufacturer_Part_Number (none) -> CL21B105KBFNNNE
- C4: Manufacturer_Part_Number (none) -> CC0805KRX7R9BB104
- D1: Manufacturer_Part_Number (none) -> SM4007PL
- D2, D3: Manufacturer_Part_Number (none) -> NCD0805R1
- F1: Manufacturer_Part_Number (none) -> BSMD1812-200-30V
- IC1: Manufacturer_Part_Number ESP32-S3-WROOM-1-N8R8 -> ESP32-S3-WROOM-1-N4
- J2: footprint TerminalBlock:TerminalBlock_bornier-3_P5.08mm -> XYEK500-5.08-3P:XYEK500-5.08-3P; Manufacturer_Part_Number (none) -> XYEK500-5.08-3P
- J6: Manufacturer_Part_Number (none) -> TYPE-C-31-M-12
- Q1: Manufacturer_Part_Number (none) -> AO3401A
- R1, R2, R6, R7: LCSC C17673 -> C17673; Manufacturer_Part_Number (none) -> 0805W8F5101T5E
- R3, R8: Manufacturer_Part_Number (none) -> 0805W8F1002T5E
- R4, R5, R9: Manufacturer_Part_Number (none) -> 0805W8F2200T5E
- SW1, SW2: Manufacturer_Part_Number (none) -> TS-1187A-B-A-B
- U1: Manufacturer_Part_Number (none) -> 0805W8F5101T5E
- U2: LCSC (none) -> C9223; Manufacturer_Part_Number (none) -> JZC-32F/005-ZS3(555)
Changed lines of the file:
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@@
+      (effects (font (size 1.27 1.27)) hide)
+    )
+    (property "Manufacturer_Part_Number" "TS-1187A-B-A-B" (at 130.81 39.37 0)
       (effects (font (size 1.27 1.27)) hide)
     )
@@
       (effects (font (size 1.27 1.27)) hide)
     )
-    (property "LCSC" " C17673" (at 116.84 64.135 0)
+    (property "LCSC" "C17673" (at 116.84 64.135 0)
+      (effects (font (size 1.27 1.27)) hide)
+    )
+    (property "Manufacturer_Part_Number" "0805W8F5101T5E" (at 116.84 64.135 0)
       (effects (font (size 1.27 1.27)) hide)
     )
@@
       (effects (font (size 1.27 1.27)) (justify left))
     )
-    (property "Footprint" "TerminalBlock:TerminalBlock_bornier-3_P5.08mm" (at 102.87 151.13 0)
+    (property "Footprint" "XYEK500-5.08-3P:XYEK500-5.08-3P" (at 102.87 151.13 0)
       (effects (font (size 1.27 1.27)) hide)
     )
     (property "Datasheet" "~" (at 102.87 151.13 0)
+      (effects (font (size 1.27 1.27)) hide)
+    )
+    (property "Manufacturer_Part_Number" "XYEK500-5.08-3P" (at 102.87 151.13 0)
       (effects (font (size 1.27 1.27)) hide)
     )
@@
       (effects (font (size 1.27 1.27)) hide)
     )
+    (property "Manufacturer_Part_Number" "0805W8F2200T5E" (at 57.15 147.32 0)
+      (effects (font (size 1.27 1.27)) hide)
+    )
     (pin "1")
     (pin "2")
@@
     )
     (property "LCSC" "C15850" (at 30.48 33.655 0)
+      (effects (font (size 1.27 1.27)) hide)
+    )
+    (property "Manufacturer_Part_Number" "CL21A106KAYNNNE" (at 30.48 33.655 0)
       (effects (font (size 1.27 1.27)) hide)
     )
@@
       (effects (font (size 1.27 1.27)) (justify left top) hide)
     )
-    (property "Manufacturer_Part_Number" "ESP32-S3-WROOM-1-N8R8" (at 172.72 824.13 0)
+    (property "Manufacturer_Part_Number" " ESP32-S3-WROOM-1-N4" (at 172.72 824.13 0)
       (effects (font (size 1.27 1.27)) (justify left top) hide)
     )
@@
       (effects (font (size 1.27 1.27)) hide)
     )
+    (property "Manufacturer_Part_Number" "CC0805KRX7R9BB104" (at 125.73 134.62 0)
+      (effects (font (size 1.27 1.27)) hide)
+    )
     (pin "1")
     (pin "2")
@@
       (effects (font (size 1.27 1.27)) hide)
     )
+    (property "LCSC" "C9223" (at 76.835 151.13 0)
+      (effects (font (size 1.27 1.27)) hide)
+    )
+    (property "Manufacturer_Part_Number" "JZC-32F/005-ZS3(555)" (at 76.835 151.13 0)
+      (effects (font (size 1.27 1.27)) hide)
+    )
     (pin "1")
     (pin "2")
@@
       (effects (font (size 1.27 1.27)) hide)
     )
+    (property "Manufacturer_Part_Number" "0805W8F2200T5E" (at 87.63 33.655 0)
+      (effects (font (size 1.27 1.27)) hide)
+    )
     (pin "1")
     (pin "2")
@@
     )
     (property "LCSC" "C318884" (at 256.54 106.68 0)
+      (effects (font (size 1.27 1.27)) hide)
+    )
+    (property "Manufacturer_Part_Number" "TS-1187A-B-A-B" (at 256.54 106.68 0)
       (effects (font (size 1.27 1.27)) hide)
     )
@@
       (effects (font (size 1.27 1.27)) hide)
     )
+    (property "Manufacturer_Part_Number" "SM4007PL" (at 73.66 152.4 0)
+      (effects (font (size 1.27 1.27)) hide)
+    )
     (pin "1")
     (pin "2")
@@
       (effects (font (size 1.27 1.27)) hide)
     )
-    (property "LCSC" " C17673" (at 57.785 62.865 0)
+    (property "LCSC" "C17673" (at 57.785 62.865 0)
+      (effects (font (size 1.27 1.27)) hide)
+    )
+    (property "Manufacturer_Part_Number" "0805W8F5101T5E" (at 57.785 62.865 0)
       (effects (font (size 1.27 1.27)) hide)
     )
@@
       (effects (font (size 1.27 1.27)) hide)
     )
+    (property "Manufacturer_Part_Number" "BSMD1812-200-30V" (at 60.325 55.245 0)
+      (effects (font (size 1.27 1.27)) hide)
+    )
     (pin "1")
     (pin "2")
@@
       (effects (font (size 1.27 1.27)) hide)
     )
-    (property "LCSC" " C17673" (at 57.785 60.325 0)
+    (property "LCSC" "C17673" (at 57.785 60.325 0)
+      (effects (font (size 1.27 1.27)) hide)
+    )
+    (property "Manufacturer_Part_Number" "0805W8F5101T5E" (at 57.785 60.325 0)
       (effects (font (size 1.27 1.27)) hide)
     )
@@
       (effects (font (size 1.27 1.27)) hide)
     )
+    (property "Manufacturer_Part_Number" "0805W8F1002T5E" (at 54.61 180.34 0)
+      (effects (font (size 1.27 1.27)) hide)
+    )
     (pin "1")
     (pin "2")
@@
       (effects (font (size 1.27 1.27)) hide)
     )
-    (property "LCSC" " C17673" (at 120.015 67.31 0)
+    (property "LCSC" "C17673" (at 120.015 67.31 0)
+      (effects (font (size 1.27 1.27)) hide)
+    )
+    (property "Manufacturer_Part_Number" "0805W8F5101T5E" (at 120.015 67.31 0)
       (effects (font (size 1.27 1.27)) hide)
     )
@@
     )
     (property "LCSC" " C165948" (at 31.115 80.645 0)
+      (effects (font (size 1.27 1.27)) hide)
+    )
+    (property "Manufacturer_Part_Number" " TYPE-C-31-M-12" (at 31.115 80.645 0)
       (effects (font (size 1.27 1.27)) hide)
     )
@@
       (effects (font (size 1.27 1.27)) hide)
     )
+    (property "Manufacturer_Part_Number" "CL21A106KAYNNNE" (at 55.88 33.655 0)
+      (effects (font (size 1.27 1.27)) hide)
+    )
     (pin "1")
     (pin "2")
@@
       (effects (font (size 1.27 1.27)) hide)
     )
+    (property "Manufacturer_Part_Number" "0805W8F2200T5E" (at 62.23 175.26 0)
+      (effects (font (size 1.27 1.27)) hide)
+    )
     (pin "1")
     (pin "2")
@@
       (effects (font (size 1.27 1.27)) hide)
     )
+    (property "Manufacturer_Part_Number" "NCD0805R1" (at 87.63 43.815 0)
+      (effects (font (size 1.27 1.27)) hide)
+    )
     (pin "1")
     (pin "2")
@@
     )
     (property "LCSC" "C28323" (at 119.38 38.1 0)
+      (effects (font (size 1.27 1.27)) hide)
+    )
+    (property "Manufacturer_Part_Number" "CL21B105KBFNNNE" (at 119.38 38.1 0)
       (effects (font (size 1.27 1.27)) hide)
     )
@@
       (effects (font (size 1.27 1.27)) hide)
     )
+    (property "Manufacturer_Part_Number" "NCD0805R1" (at 57.15 156.21 0)
+      (effects (font (size 1.27 1.27)) hide)
+    )
     (pin "1")
     (pin "2")
@@
       (effects (font (size 1.27 1.27)) hide)
     )
+    (property "Manufacturer_Part_Number" "0805W8F1002T5E" (at 113.03 34.29 0)
+      (effects (font (size 1.27 1.27)) hide)
+    )
     (pin "1")
     (pin "2")
@@
       (effects (font (size 1.27 1.27)) hide)
     )
+    (property "Manufacturer_Part_Number" "AO3401A" (at 71.12 175.26 0)
+      (effects (font (size 1.27 1.27)) hide)
+    )
     (pin "1")
     (pin "2")
@@
       (effects (font (size 1.27 1.27)) hide)
     )
+    (property "Manufacturer_Part_Number" "0805W8F5101T5E" (at 43.18 27.94 0)
+      (effects (font (size 1.27 1.27)) hide)
+    )
