File: board-clima-esp32.kicad_sch (KiCad schematic)
At the start: 57 parts, among them IC1 ESP32-S3-WROOM-1-N4, J1 Conn_01x06_Pin, J2 Screw_Terminal_01x03, J3 Conn_01x04_Pin, J4 Screw_Terminal_01x02, J5 Conn_01x05_Pin, J6 USB_C_Receptacle, Q1 AO3400A, Q2 AO3401A, Q3 AO3400A, SW1 RESET, SW2 BOOT, U1 AMS1117-3.3, U3 PC817, U4 PC817

Commit message: final corrections
Parts:
- added TP1, TP2, TP3, TP4, TP5, TP6: TestPoint, TestPoint:TestPoint_Pad_D1.0mm, symbol Connector:TestPoint
Connections:
- net BOILER_1: now also TP1.1
- net BOILER_2: now also TP2.1
- net at IC1.32 (IO39): now also TP3.1
- net at IC1.33 (IO40): now also TP4.1
- net at IC1.34 (IO41): now also TP5.1
- net at IC1.35 (IO42): now also TP6.1
- no-connect marks 35 -> 31
Other:
- note added: "EMERGENCY JTAG"
Changed lines of the file:
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@@
   (junction (at 194.31 34.29) (diameter 0) (color 0 0 0 0)
   )
+  (junction (at 189.23 74.93) (diameter 0) (color 0 0 0 0)
+  )
   (junction (at 240.03 67.31) (diameter 0) (color 0 0 0 0)
   )
@@
   (junction (at 200.66 25.4) (diameter 0) (color 0 0 0 0)
   )
+  (junction (at 186.69 72.39) (diameter 0) (color 0 0 0 0)
+  )
   (junction (at 186.69 87.63) (diameter 0) (color 0 0 0 0)
   )
@@
   (no_connect (at 207.01 41.91))
   (no_connect (at 207.01 39.37))
-  (no_connect (at 240.03 52.07))
   (no_connect (at 45.72 64.77))
   (no_connect (at 45.72 59.69))
-  (no_connect (at 240.03 46.99))
   (no_connect (at 240.03 39.37))
   (no_connect (at 45.72 57.15))
@@
   (no_connect (at 45.72 82.55))
   (no_connect (at 240.03 34.29))
-  (no_connect (at 240.03 44.45))
   (no_connect (at 45.72 67.31))
   (no_connect (at 240.03 29.21))
@@
   (no_connect (at 207.01 49.53))
   (no_connect (at 207.01 54.61))
-  (no_connect (at 240.03 49.53))
   (no_connect (at 207.01 69.85))
   (no_connect (at 207.01 52.07))
@@
     (stroke (width 0) (type default))
   )
+  (wire (pts (xy 189.23 71.12) (xy 189.23 74.93))
+    (stroke (width 0) (type default))
+  )
   (wire (pts (xy 254 120.65) (xy 260.35 120.65))
     (stroke (width 0) (type default))
@@
     (stroke (width 0) (type default))
   )
-  (wire (pts (xy 173.99 74.93) (xy 207.01 74.93))
+  (wire (pts (xy 173.99 74.93) (xy 189.23 74.93))
     (stroke (width 0) (type default))
   )
@@
     (stroke (width 0) (type default))
   )
-  (wire (pts (xy 173.99 72.39) (xy 207.01 72.39))
+  (wire (pts (xy 173.99 72.39) (xy 186.69 72.39))
     (stroke (width 0) (type default))
   )
@@
     (stroke (width 0) (type default))
   )
+  (wire (pts (xy 189.23 74.93) (xy 207.01 74.93))
+    (stroke (width 0) (type default))
+  )
   (wire (pts (xy 381 77.47) (xy 387.35 77.47))
     (stroke (width 0) (type default))
@@
     (stroke (width 0) (type default))
   )
+  (wire (pts (xy 186.69 72.39) (xy 207.01 72.39))
+    (stroke (width 0) (type default))
+  )
   (wire (pts (xy 335.28 62.23) (xy 335.28 73.66))
     (stroke (width 0) (type default))
@@
     (stroke (width 0) (type default))
   )
+  (wire (pts (xy 186.69 71.12) (xy 186.69 72.39))
+    (stroke (width 0) (type default))
+  )
   (wire (pts (xy 182.88 85.09) (xy 207.01 85.09))
     (stroke (width 0) (type default))
@@
     (effects (font (size 1.27 1.27)) (justify left bottom))
   )
+  (text "EMERGENCY\nJTAG" (at 248.92 50.8 0)
+    (effects (font (size 1.27 1.27)) (justify left bottom))
+  )
   (text "Boot\nSelector" (at 157.48 41.275 0)
     (effects (font (size 1.27 1.27)) (justify left bottom))
@@
     )
   )
+  (symbol (lib_id "Connector:TestPoint") (at 240.03 52.07 270) (unit 1)
+    (in_bom yes) (on_board yes) (dnp no)
+    (property "Reference" "TP6" (at 243.84 52.07 90)
+      (effects (font (size 1.27 1.27)) (justify left))
+    )
+    (property "Value" "TestPoint" (at 245.11 53.34 90)
+      (effects (font (size 1.27 1.27)) (justify left) hide)
+    )
+    (property "Footprint" "TestPoint:TestPoint_Pad_D1.0mm" (at 240.03 57.15 0)
+      (effects (font (size 1.27 1.27)) hide)
+    )
+    (property "Datasheet" "~" (at 240.03 57.15 0)
+      (effects (font (size 1.27 1.27)) hide)
+    )
+    (pin "1")
+    (instances
+      (project "board-clima-esp32"
+        (path "/ec184202-d4fa-4f1f-9fe7-c32d14dd4c20"
+          (reference "TP6") (unit 1)
+        )
+      )
+    )
+  )
   (symbol (lib_id "Device:R") (at 46.99 158.75 270) (unit 1)
     (in_bom yes) (on_board yes) (dnp no)
@@
     )
   )
+  (symbol (lib_id "Connector:TestPoint") (at 240.03 49.53 270) (unit 1)
+    (in_bom yes) (on_board yes) (dnp no)
+    (property "Reference" "TP5" (at 243.84 49.53 90)
+      (effects (font (size 1.27 1.27)) (justify left))
+    )
+    (property "Value" "TestPoint" (at 245.11 50.8 90)
+      (effects (font (size 1.27 1.27)) (justify left) hide)
+    )
+    (property "Footprint" "TestPoint:TestPoint_Pad_D1.0mm" (at 240.03 54.61 0)
+      (effects (font (size 1.27 1.27)) hide)
+    )
+    (property "Datasheet" "~" (at 240.03 54.61 0)
+      (effects (font (size 1.27 1.27)) hide)
+    )
+    (pin "1")
+    (instances
+      (project "board-clima-esp32"
+        (path "/ec184202-d4fa-4f1f-9fe7-c32d14dd4c20"
+          (reference "TP5") (unit 1)
+        )
+      )
+    )
+  )
   (symbol (lib_id "Mechanical:MountingHole") (at 373.38 221.615 0) (unit 1)
     (in_bom yes) (on_board yes) (dnp no) (fields_autoplaced)
@@
     )
   )
+  (symbol (lib_id "Connector:TestPoint") (at 240.03 46.99 270) (unit 1)
+    (in_bom yes) (on_board yes) (dnp no)
+    (property "Reference" "TP4" (at 243.84 46.99 90)
+      (effects (font (size 1.27 1.27)) (justify left))
+    )
+    (property "Value" "TestPoint" (at 245.11 48.26 90)
+      (effects (font (size 1.27 1.27)) (justify left) hide)
+    )
+    (property "Footprint" "TestPoint:TestPoint_Pad_D1.0mm" (at 240.03 52.07 0)
+      (effects (font (size 1.27 1.27)) hide)
+    )
+    (property "Datasheet" "~" (at 240.03 52.07 0)
+      (effects (font (size 1.27 1.27)) hide)
+    )
+    (pin "1")
+    (instances
+      (project "board-clima-esp32"
+        (path "/ec184202-d4fa-4f1f-9fe7-c32d14dd4c20"
+          (reference "TP4") (unit 1)
+        )
+      )
+    )
+  )
   (symbol (lib_id "Device:R") (at 57.15 29.21 90) (unit 1)
     (in_bom yes) (on_board yes) (dnp no)
@@
     )
   )
+  (symbol (lib_id "Connector:TestPoint") (at 189.23 71.12 0) (unit 1)
+    (in_bom yes) (on_board yes) (dnp no)
+    (property "Reference" "TP2" (at 189.23 66.04 0)
+      (effects (font (size 1.27 1.27)) (justify left))
+    )
+    (property "Value" "TestPoint" (at 191.77 69.088 0)
+      (effects (font (size 1.27 1.27)) (justify left) hide)
+    )
+    (property "Footprint" "TestPoint:TestPoint_Pad_D1.0mm" (at 194.31 71.12 0)
+      (effects (font (size 1.27 1.27)) hide)
+    )
+    (property "Datasheet" "~" (at 194.31 71.12 0)
+      (effects (font (size 1.27 1.27)) hide)
+    )
+    (pin "1")
+    (instances
+      (project "board-clima-esp32"
+        (path "/ec184202-d4fa-4f1f-9fe7-c32d14dd4c20"
+          (reference "TP2") (unit 1)
+        )
+      )
+    )
+  )
   (symbol (lib_id "Mechanical:MountingHole") (at 373.38 234.95 0) (unit 1)
     (in_bom yes) (on_board yes) (dnp no) (fields_autoplaced)
@@
     )
   )
+  (symbol (lib_id "Connector:TestPoint") (at 240.03 44.45 270) (unit 1)
+    (in_bom yes) (on_board yes) (dnp no)
+    (property "Reference" "TP3" (at 243.84 44.45 90)
+      (effects (font (size 1.27 1.27)) (justify left))
+    )
+    (property "Value" "TestPoint" (at 245.11 45.72 90)
+      (effects (font (size 1.27 1.27)) (justify left) hide)
+    )
+    (property "Footprint" "TestPoint:TestPoint_Pad_D1.0mm" (at 240.03 49.53 0)
+      (effects (font (size 1.27 1.27)) hide)
+    )
+    (property "Datasheet" "~" (at 240.03 49.53 0)
+      (effects (font (size 1.27 1.27)) hide)
+    )
+    (pin "1")
+    (instances
+      (project "board-clima-esp32"
+        (path "/ec184202-d4fa-4f1f-9fe7-c32d14dd4c20"
+          (reference "TP3") (unit 1)
+        )
+      )
+    )
+  )
   (symbol (lib_id "Connector:Screw_Terminal_01x03") (at 400.05 62.23 0) (unit 1)
     (in_bom yes) (on_board yes) (dnp no)
@@
         )
       )
+    )
+  )
+  (symbol (lib_id "Connector:TestPoint") (at 186.69 71.12 0) (unit 1)
+    (in_bom yes) (on_board yes) (dnp no)
+    (property "Reference" "TP1" (at 182.88 66.04 0)
+      (effects (font (size 1.27 1.27)) (justify left))
+    )
+    (property "Value" "TestPoint" (at 189.23 69.088 0)
+      (effects (font (size 1.27 1.27)) (justify left) hide)
+    )
+    (property "Footprint" "TestPoint:TestPoint_Pad_D1.0mm" (at 191.77 71.12 0)
+      (effects (font (size 1.27 1.27)) hide)
+    )
+    (property "Datasheet" "~" (at 191.77 71.12 0)
+      (effects (font (size 1.27 1.27)) hide)
+    )
+    (pin "1")
+    (instances
+      (project "board-clima-esp32"
+        (path "/ec184202-d4fa-4f1f-9fe7-c32d14dd4c20"
+          (reference "TP1") (unit 1)
+        )
+      )

Commit message: drc pass
Other:
- note added: "OT RX"
- note added: "OT TX"
Changed lines of the file:
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@@
     (stroke (width 0) (type default))
   )
-  (wire (pts (xy 248.92 146.05) (xy 248.92 142.24))
+  (wire (pts (xy 250.19 146.05) (xy 250.19 142.24))
     (stroke (width 0) (type default))
   )
@@
     (stroke (width 0) (type default))
   )
-  (wire (pts (xy 245.11 146.05) (xy 248.92 146.05))
+  (wire (pts (xy 245.11 146.05) (xy 250.19 146.05))
     (stroke (width 0) (type default))
   )
@@
     (effects (font (size 2 2) (thickness 0.4) bold) (justify left bottom))
   )
+  (text "OT TX" (at 234.95 118.11 0)
+    (effects (font (size 1.27 1.27)) (justify left bottom))
+  )
   (text "Temperature Sensor" (at 307.34 85.09 0)
     (effects (font (size 1.27 1.27)) (justify left bottom))
@@
   (text "PSRAM" (at 241.3 39.37 0)
     (effects (font (size 1.27 1.27) (color 255 0 0 1)) (justify left bottom))
+  )
+  (text "OT RX" (at 234.95 143.51 0)
+    (effects (font (size 1.27 1.27)) (justify left bottom))
   )
   (text "Power" (at 80.01 101.6 0)
@@
     )
   )
-  (symbol (lib_id "power:+3.3V") (at 248.92 142.24 0) (unit 1)
-    (in_bom yes) (on_board yes) (dnp no) (fields_autoplaced)
-    (property "Reference" "#PWR030" (at 248.92 146.05 0)
-      (effects (font (size 1.27 1.27)) hide)
-    )
-    (property "Value" "+3.3V" (at 248.92 137.795 0)
-      (effects (font (size 1.27 1.27)))
-    )
-    (property "Footprint" "" (at 248.92 142.24 0)
-      (effects (font (size 1.27 1.27)) hide)
-    )
-    (property "Datasheet" "" (at 248.92 142.24 0)
-      (effects (font (size 1.27 1.27)) hide)
-    )
+  (symbol (lib_id "power:+3.3V") (at 250.19 142.24 0) (unit 1)
+    (in_bom yes) (on_board yes) (dnp no) (fields_autoplaced)
+    (property "Reference" "#PWR030" (at 250.19 146.05 0)
+      (effects (font (size 1.27 1.27)) hide)
+    )
+    (property "Value" "+3.3V" (at 250.19 137.795 0)
+      (effects (font (size 1.27 1.27)))
+    )
+    (property "Footprint" "" (at 250.19 142.24 0)
+      (effects (font (size 1.27 1.27)) hide)
+    )
+    (property "Datasheet" "" (at 250.19 142.24 0)
+      (effects (font (size 1.27 1.27)) hide)
+    )
